Commit message: Adjusts joint limits and adds gripper visualization
Updates robot joint effort limits and range constraints to match real hardware specs:
- Reduces joint 1 range to ±1.6 rad and increases effort to 40
- Adjusts effort limits for other joints for better control
- Adds gripper visualization link for improved monitoring

Switches default control mode to joint torque control
Updates initial robot pose to have proper Z-height

File: assets/urdf/ino_ir_400_4/urdf/ino_ir_400_4.urdf (robot description, URDF)
Before this commit: robot ino_ir_400_4, 17 links, 16 joints
Links:
- added link grip_site; visual sphere radius=0.001
- link cam_point: geometry visual sphere radius=0.001
Joints:
- added joint grip_vis_joint: type fixed, parent hand_base_link, child grip_site, origin xyz=0.0408 0 -0.2661 rpy=0 0 0
- joint joint1: limit lower=-2.3038 upper=2.3038 effort=1 velocity=6.2832 -> lower=-1.6 upper=1.6 effort=40 velocity=6.2832
- joint joint2: limit lower=-2.4609 upper=2.4609 effort=1 velocity=6.2832 -> lower=-2.4609 upper=2.4609 effort=30 velocity=6.2832
- joint joint3: limit lower=-0.04 upper=0 effort=100 velocity=1.3 -> lower=-0.04 upper=0 effort=20 velocity=1.3
- joint joint4: limit lower=-3.1416 upper=3.1416 effort=1 velocity=45.379 -> lower=-1.1416 upper=1.1416 effort=10 velocity=45.379
